File: LED grid 8x8.kicad_pcb (KiCad board)
At the start: 2 copper layers, 68.6 x 53.3 mm, 11 parts, among them P1 Power, P2 Analog, P3 Digital, P4 Digital, P5 CONN_1, P6 CONN_1, P7 CONN_1, P8 CONN_1, U1 74HC595, U2 74HC595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

Commit message: added front silk on pcb
Other:
- board text added: "Marginallyclever.com 2017-3-8 shift register LED grid"
Changed lines of the file:
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@@
     (area 110.922999 72.949999 179.653001 126.440001)
     (thickness 1.6)
-    (drawings 27)
+    (drawings 28)
     (tracks 61)
     (zones 0)
@@
       (net 42 "Net-(U1-Pad7)"))
   )
+  (gr_text "Marginallyclever.com 2017-3-8\nshift register LED grid" (at 115.57 102.489 90) (layer F.SilkS)
+    (effects (font (size 1.5 1.5) (thickness 0.3)))
+  )
   (gr_text 1 (at 138.938 121.285 90) (layer F.SilkS)
